Commit message: Updated Dobot MoveIt config and trajectory bridge

File: src/dobot_moveit_config/config/dobot.urdf.xacro (robot description, xacro)
@@ -1,4 +1,4 @@
 <?xml version="1.0"?>
-<robot name="dobot">
+<robot name="dobot_magician">
   <!-- ================= BASE ================= -->
   <link name="base_link">
@@ -13,5 +13,5 @@
   </link>
   <!-- ================= LINK 1 ================= -->
-  <link name="link1">
+  <link name="magician_link_1">
     <visual>
       <origin xyz="0 0 0.05" rpy="0 0 0"/>
@@ -25,5 +25,5 @@
   </link>
   <!-- ================= LINK 2 ================= -->
-  <link name="link2">
+  <link name="magician_link_2">
     <visual>
       <origin xyz="0 0 0.10" rpy="0 0 0"/>
@@ -37,5 +37,5 @@
   </link>
   <!-- ================= LINK 3 ================= -->
-  <link name="link3">
+  <link name="magician_link_3">
     <visual>
       <origin xyz="0 0 0.08" rpy="0 0 0"/>
@@ -49,5 +49,5 @@
   </link>
   <!-- ================= LINK 4 (WRIST) ================= -->
-  <link name="link4">
+  <link name="magician_link_4">
     <visual>
       <origin xyz="0 0 0.03" rpy="0 0 0"/>
@@ -81,5 +81,5 @@
   <joint name="joint1" type="revolute">
     <parent link="base_link"/>
-    <child link="link1"/>
+    <child link="magician_link_1"/>
     <origin xyz="0 0 0.05" rpy="0 0 0"/>
     <axis xyz="0 0 1"/>
@@ -87,6 +87,6 @@
   </joint>
   <joint name="joint2" type="revolute">
-    <parent link="link1"/>
-    <child link="link2"/>
+    <parent link="magician_link_1"/>
+    <child link="magician_link_2"/>
     <origin xyz="0 0 0.10" rpy="0 0 0"/>
     <axis xyz="0 1 0"/>
@@ -94,6 +94,6 @@
   </joint>
   <joint name="joint3" type="revolute">
-    <parent link="link2"/>
-    <child link="link3"/>
+    <parent link="magician_link_2"/>
+    <child link="magician_link_3"/>
     <origin xyz="0 0 0.20" rpy="0 0 0"/>
     <axis xyz="0 1 0"/>
@@ -101,6 +101,6 @@
   </joint>
   <joint name="joint4" type="revolute">
-    <parent link="link3"/>
-    <child link="link4"/>
+    <parent link="magician_link_3"/>
+    <child link="magician_link_4"/>
     <origin xyz="0 0 0.16" rpy="0 0 0"/>
     <axis xyz="0 0 1"/>
@@ -109,5 +109,5 @@
   <!-- ================= FIXED TOOL JOINT ================= -->
   <joint name="tool0_fixed_joint" type="fixed">
-    <parent link="link4"/>
+    <parent link="magician_link_4"/>
     <child link="tool0"/>
     <origin xyz="0 0 0.06" rpy="0 0 0"/>

File: src/robot_description/urdf/dobot.urdf.xacro (robot description, xacro)
@@ -1,4 +1,4 @@
 <?xml version="1.0"?>
-<robot name="dobot" xmlns:xacro="http://www.ros.org/wiki/xacro">
+<robot name="dobot_magician" xmlns:xacro="http://www.ros.org/wiki/xacro">
   <!-- ================= BASE ================= -->
   <link name="base_link">
@@ -24,5 +24,5 @@
   <joint name="joint1" type="revolute">
     <parent link="base_link"/>
-    <child link="link1"/>
+    <child link="magician_link_1"/>
     <origin xyz="0 0 0.03" rpy="0 0 0"/>
     <axis xyz="0 0 1"/>
@@ -30,5 +30,5 @@
   </joint>
   <!-- ================= LINK 1 ================= -->
-  <link name="link1">
+  <link name="magician_link_1">
     <visual>
       <geometry>
@@ -51,6 +51,6 @@
   <!-- ================= JOINT 2 ================= -->
   <joint name="joint2" type="revolute">
-    <parent link="link1"/>
-    <child link="link2"/>
+    <parent link="magician_link_1"/>
+    <child link="magician_link_2"/>
     <origin xyz="0.12 0 0" rpy="0 0 0"/>
     <axis xyz="0 1 0"/>
@@ -58,5 +58,5 @@
   </joint>
   <!-- ================= LINK 2 ================= -->
-  <link name="link2">
+  <link name="magician_link_2">
     <visual>
       <geometry>
@@ -79,6 +79,6 @@
   <!-- ================= JOINT 3 ================= -->
   <joint name="joint3" type="revolute">
-    <parent link="link2"/>
-    <child link="link3"/>
+    <parent link="magician_link_2"/>
+    <child link="magician_link_3"/>
     <origin xyz="0.14 0 0" rpy="0 0 0"/>
     <axis xyz="0 1 0"/>
@@ -86,5 +86,5 @@
   </joint>
   <!-- ================= LINK 3 ================= -->
-  <link name="link3">
+  <link name="magician_link_3">
     <visual>
       <geometry>
@@ -107,5 +107,5 @@
   <!-- ================= JOINT 4 ================= -->
   <joint name="joint4" type="revolute">
-    <parent link="link3"/>
+    <parent link="magician_link_3"/>
     <child link="tool0"/>
     <origin xyz="0.10 0 0" rpy="0 0 0"/>
