Commit message: Integrated Dobot ros2_control hardware, MoveIt2 configs, and controller updates

File: src/dobot_moveit_config/config/dobot.ros2_control.xacro (robot description, xacro)
@@ -1,40 +1,24 @@
 <?xml version="1.0"?>
 <robot xmlns:xacro="http://www.ros.org/wiki/xacro">
-    <xacro:macro name="dobot_ros2_control" params="name initial_positions_file">
-        <xacro:property name="initial_positions" value="${xacro.load_yaml(initial_positions_file)['initial_positions']}"/>
-        <ros2_control name="${name}" type="system">
-            <hardware>
-                <!-- By default, set up controllers for simulation. This won't work on real hardware -->
-                <plugin>mock_components/GenericSystem</plugin>
-            </hardware>
-            <joint name="joint1">
-                <command_interface name="position"/>
-                <state_interface name="position">
-                  <param name="initial_value">${initial_positions['joint1']}</param>
-                </state_interface>
-                <state_interface name="velocity"/>
-            </joint>
-            <joint name="joint2">
-                <command_interface name="position"/>
-                <state_interface name="position">
-                  <param name="initial_value">${initial_positions['joint2']}</param>
-                </state_interface>
-                <state_interface name="velocity"/>
-            </joint>
-            <joint name="joint3">
-                <command_interface name="position"/>
-                <state_interface name="position">
-                  <param name="initial_value">${initial_positions['joint3']}</param>
-                </state_interface>
-                <state_interface name="velocity"/>
-            </joint>
-            <joint name="joint4">
-                <command_interface name="position"/>
-                <state_interface name="position">
-                  <param name="initial_value">${initial_positions['joint4']}</param>
-                </state_interface>
-                <state_interface name="velocity"/>
-            </joint>
-        </ros2_control>
-    </xacro:macro>
+  <ros2_control name="DobotSystem" type="system">
+    <hardware>
+      <plugin>dobot_hardware/DobotHardware</plugin>
+    </hardware>
+    <joint name="joint1">
+      <command_interface name="position"/>
+      <state_interface name="position"/>
+    </joint>
+    <joint name="joint2">
+      <command_interface name="position"/>
+      <state_interface name="position"/>
+    </joint>
+    <joint name="joint3">
+      <command_interface name="position"/>
+      <state_interface name="position"/>
+    </joint>
+    <joint name="joint4">
+      <command_interface name="position"/>
+      <state_interface name="position"/>
+    </joint>
+  </ros2_control>
 </robot>

File: src/dobot_moveit_config/config/dobot.urdf.xacro (robot description, xacro)
@@ -1,9 +1,137 @@
 <?xml version="1.0"?>
-<robot xmlns:xacro="http://www.ros.org/wiki/xacro" name="dobot">
-    <xacro:arg name="initial_positions_file" default="initial_positions.yaml" />
-    <!-- Import dobot urdf file -->
-    <xacro:include filename="/home/anagha/robot_control_ws/src/robot_description/urdf/dobot.urdf.xacro" />
-    <!-- Import control_xacro -->
-    <xacro:include filename="dobot.ros2_control.xacro" />
-    <xacro:dobot_ros2_control name="FakeSystem" initial_positions_file="$(arg initial_positions_file)"/>
+<robot name="dobot">
+  <!-- ================= BASE ================= -->
+  <link name="base_link">
+    <visual>
+      <geometry>
+        <box size="0.12 0.12 0.05"/>
+      </geometry>
+      <material name="grey">
+        <color rgba="0.6 0.6 0.6 1"/>
+      </material>
+    </visual>
+  </link>
+  <!-- ================= LINK 1 ================= -->
+  <link name="link1">
+    <visual>
+      <origin xyz="0 0 0.05" rpy="0 0 0"/>
+      <geometry>
+        <cylinder radius="0.02" length="0.10"/>
+      </geometry>
+      <material name="blue">
+        <color rgba="0 0 1 1"/>
+      </material>
+    </visual>
+  </link>
+  <!-- ================= LINK 2 ================= -->
+  <link name="link2">
+    <visual>
+      <origin xyz="0 0 0.10" rpy="0 0 0"/>
+      <geometry>
+        <cylinder radius="0.02" length="0.20"/>
+      </geometry>
+      <material name="green">
+        <color rgba="0 1 0 1"/>
+      </material>
+    </visual>
+  </link>
+  <!-- ================= LINK 3 ================= -->
+  <link name="link3">
+    <visual>
+      <origin xyz="0 0 0.08" rpy="0 0 0"/>
+      <geometry>
+        <cylinder radius="0.015" length="0.16"/>
+      </geometry>
+      <material name="red">
+        <color rgba="1 0 0 1"/>
+      </material>
+    </visual>
+  </link>
+  <!-- ================= LINK 4 (WRIST) ================= -->
+  <link name="link4">
+    <visual>
+      <origin xyz="0 0 0.03" rpy="0 0 0"/>
+      <geometry>
+        <sphere radius="0.02"/>
+      </geometry>
+      <material name="cyan">
+        <color rgba="0 1 1 1"/>
+      </material>
+    </visual>
+  </link>
+  <!-- ================= TOOL LINK ================= -->
+  <link name="tool0">
+    <visual>
+      <origin xyz="0 0 0.025" rpy="0 0 0"/>
+      <geometry>
+        <cylinder radius="0.015" length="0.05"/>
+      </geometry>
+      <material name="black">
+        <color rgba="0.1 0.1 0.1 1"/>
+      </material>
+    </visual>
+    <collision>
+      <origin xyz="0 0 0.025" rpy="0 0 0"/>
+      <geometry>
+        <cylinder radius="0.015" length="0.05"/>
+      </geometry>
+    </collision>
+  </link>
+  <!-- ================= JOINTS ================= -->
+  <joint name="joint1" type="revolute">
+    <parent link="base_link"/>
+    <child link="link1"/>
+    <origin xyz="0 0 0.05" rpy="0 0 0"/>
+    <axis xyz="0 0 1"/>
+    <limit lower="-3.14" upper="3.14" effort="10" velocity="1.0"/>
+  </joint>
+  <joint name="joint2" type="revolute">
+    <parent link="link1"/>
+    <child link="link2"/>
+    <origin xyz="0 0 0.10" rpy="0 0 0"/>
+    <axis xyz="0 1 0"/>
+    <limit lower="-1.57" upper="1.57" effort="10" velocity="1.0"/>
+  </joint>
+  <joint name="joint3" type="revolute">
+    <parent link="link2"/>
+    <child link="link3"/>
+    <origin xyz="0 0 0.20" rpy="0 0 0"/>
+    <axis xyz="0 1 0"/>
+    <limit lower="-1.57" upper="1.57" effort="10" velocity="1.0"/>
+  </joint>
+  <joint name="joint4" type="revolute">
+    <parent link="link3"/>
+    <child link="link4"/>
+    <origin xyz="0 0 0.16" rpy="0 0 0"/>
+    <axis xyz="0 0 1"/>
+    <limit lower="-3.14" upper="3.14" effort="10" velocity="1.0"/>
+  </joint>
+  <!-- ================= FIXED TOOL JOINT ================= -->
+  <joint name="tool0_fixed_joint" type="fixed">
+    <parent link="link4"/>
+    <child link="tool0"/>
+    <origin xyz="0 0 0.06" rpy="0 0 0"/>
+  </joint>
+  <!-- ================= ros2_control ================= -->
+  <ros2_control name="DobotSystem" type="system">
+    <hardware>
+      <plugin>dobot_hardware/DobotHardware</plugin>
+    </hardware>
+    <joint name="joint1">
+      <command_interface name="position"/>
+      <state_interface name="position"/>
+    </joint>
+    <joint name="joint2">
+      <command_interface name="position"/>
+      <state_interface name="position"/>
+    </joint>
+    <joint name="joint3">
+      <command_interface name="position"/>
+      <state_interface name="position"/>
+    </joint>
+    <joint name="joint4">
+      <command_interface name="position"/>
+      <state_interface name="position"/>
+    </joint>
+  </ros2_control>
 </robot>

Commit message: Initial ROS2 workspace for Dobot Magician Lite

File: src/dobot_moveit_config/config/dobot.ros2_control.xacro (robot description, xacro)
@@ -4,18 +4,31 @@
     <hardware>
       <plugin>dobot_hardware/DobotHardware</plugin>
+      <param name="port">/dev/ttyACM0</param>
+      <param name="baudrate">115200</param>
+      <param name="dof">4</param>
     </hardware>
-    <joint name="joint1">
+    <!-- Arm joints -->
+    <joint name="magician_joint_1">
       <command_interface name="position"/>
       <state_interface name="position"/>
     </joint>
-    <joint name="joint2">
+    <joint name="magician_joint_2">
       <command_interface name="position"/>
       <state_interface name="position"/>
     </joint>
-    <joint name="joint3">
+    <joint name="magician_joint_3">
       <command_interface name="position"/>
       <state_interface name="position"/>
     </joint>
-    <joint name="joint4">
+    <joint name="magician_joint_4">
+      <command_interface name="position"/>
+      <state_interface name="position"/>
+    </joint>
+    <!-- Gripper (optional, but included for completeness) -->
+    <joint name="magician_joint_prismatic_l">
+      <command_interface name="position"/>
+      <state_interface name="position"/>
+    </joint>
+    <joint name="magician_joint_prismatic_r">
       <command_interface name="position"/>
       <state_interface name="position"/>

File: src/dobot_moveit_config/config/dobot.urdf.xacro (robot description, xacro)
@@ -2,5 +2,5 @@
 <robot name="dobot_magician">
   <!-- ================= BASE ================= -->
-  <link name="base_link">
+  <link name="magician_base_link">
     <visual>
       <geometry>
@@ -79,6 +79,6 @@
   </link>
   <!-- ================= JOINTS ================= -->
-  <joint name="joint1" type="revolute">
-    <parent link="base_link"/>
+  <joint name="magician_joint_1" type="revolute">
+    <parent link="magician_base_link"/>
     <child link="magician_link_1"/>
     <origin xyz="0 0 0.05" rpy="0 0 0"/>
@@ -86,5 +86,5 @@
     <limit lower="-3.14" upper="3.14" effort="10" velocity="1.0"/>
   </joint>
-  <joint name="joint2" type="revolute">
+  <joint name="magician_joint_2" type="revolute">
     <parent link="magician_link_1"/>
     <child link="magician_link_2"/>
@@ -93,5 +93,5 @@
     <limit lower="-1.57" upper="1.57" effort="10" velocity="1.0"/>
   </joint>
-  <joint name="joint3" type="revolute">
+  <joint name="magician_joint_3" type="revolute">
     <parent link="magician_link_2"/>
     <child link="magician_link_3"/>
@@ -100,5 +100,5 @@
     <limit lower="-1.57" upper="1.57" effort="10" velocity="1.0"/>
   </joint>
-  <joint name="joint4" type="revolute">
+  <joint name="magician_joint_4" type="revolute">
     <parent link="magician_link_3"/>
     <child link="magician_link_4"/>
@@ -118,17 +118,17 @@
       <plugin>dobot_hardware/DobotHardware</plugin>
     </hardware>
-    <joint name="joint1">
+    <joint name="magician_joint_1">
       <command_interface name="position"/>
       <state_interface name="position"/>
     </joint>
-    <joint name="joint2">
+    <joint name="magician_joint_2">
       <command_interface name="position"/>
       <state_interface name="position"/>
     </joint>
-    <joint name="joint3">
+    <joint name="magician_joint_3">
       <command_interface name="position"/>
       <state_interface name="position"/>
     </joint>
-    <joint name="joint4">
+    <joint name="magician_joint_4">
       <command_interface name="position"/>
       <state_interface name="position"/>
